File: led_board.kicad_sch (KiCad schematic)
At the start: 193 parts, among them J1 SEAM-50-01-L-06-2-RA-GP-TR

Commit message: first prod ver, with well plate mount
Parts:
- added H1, H2, H3: MountingHole_Pad, MountingHole:MountingHole_3.5mm_Pad_TopBottom, symbol Mechanical:MountingHole_Pad
- D100, D101, D102, D103, D104, D105, D106, D107, D108, D109, D110, D111, D112, D113, D114, D115, D116, D117, D118, D119, D120, D121, D122, D123, D124, D125, D126, D127, D128, D129, D130, D131, D132, D133, D134, D135, D136, D137, D138, D139, D140, D141, D142, D143, D144, D145, D146, D147, D148, D149, D150, D151, D152, D153, D154, D155, D156, D157, D158, D159, D160, D161, D162, D163, D164, D165, D166, D167, D168, D169, D170, D171, D172, D173, D174, D175, D176, D177, D178, D179, D180, D181, D182, D183, D184, D185, D186, D187, D188, D189, D190, D191, D192, D97, D98, D99: footprint LED_SMD:GFJTLPS124KXK511 -> GF_JTLP mod:GFJTLPS124KXK511
Connections:
- net GND: now also H1.1, H2.1, H3.1
Other:
- moved on the sheet: J1B, J1C
